Commit message: [add] 並行チャックのモデルを追加

File: motoman_description/urdf/common.xacro (robot description, xacro)
@@ -1,4 +1,20 @@
 <?xml version="1.0"?>
-<robot>
+<robot xmlns:xacro="http://ros.org/wiki/xacro>">
   <property name="M_PI" value="3.14159274"/>
+  <xacro:macro name="cylinder_inertial" params="mass radius length">
+	<inertial>
+	  <mass value="${mass}"/>
+	  <inertia ixx="${((radius*radius)/4 + (length*length)/12)*mass}" ixy="0" ixz="0"
+			   iyy="${((radius*radius)/4 + (length*length)/12)*mass}" iyz="0"
+			   izz="${(mass*radius*radius)/2}" />
+	</inertial>
+  </xacro:macro>
+  <xacro:macro name="box_inertial" params="mass height width depth">
+	<inertial>
+	  <mass value="${mass}"/>
+	  <inertia ixx="${(mass*(width*width+depth*depth))/12}" ixy="0" ixz="0"
+			   iyy="${(mass*(height*height+depth*depth))/12}" iyz="0"
+			   izz="${(mass*(height*height+width*width))/12}" />
+	</inertial>
+  </xacro:macro>
 </robot>
