Commit message: [fix] collision情報を修正

File: motoman_description/urdf/tool/parallel/parallel.urdf.xacro (robot description, xacro)
@@ -45,5 +45,5 @@
 	  <collision>
 		<geometry>
-		  <box size="0.025 0.05 0.1"/>
+		  <box size="0.1 0.025 0.025"/>
 		</geometry>
 	  </collision>

Commit message: [modify] トルクリミットを変更

File: motoman_description/urdf/tool/parallel/parallel.urdf.xacro (robot description, xacro)
@@ -34,5 +34,5 @@
 	  <parent link="parallel_base_link"/>
 	  <child link="parallel_${prefix}_grip_link"/>
-	  <limit lower="0" upper="0.05" effort="0.5" velocity="6.0" />
+	  <limit lower="0" upper="0.05" effort="100" velocity="100" />
 	</joint>
 	<link name="parallel_${prefix}_grip_link">
