Commit message: [modify] ロボットを床から浮かせた

File: motoman_description/robots/sia5/sia5_with_parallel.urdf.xacro (robot description, xacro)
@@ -3,5 +3,8 @@
   <!-- File Include -->
   <xacro:include filename="$(find motoman_description)/urdf/tool/parallel/parallel.urdf.xacro"/>
-  <xacro:include filename="$(find motoman_description)/robots/sia5/sia5.urdf.xacro"/>
+  <xacro:include filename="$(find motoman_description)/robots/sia5/sia5_basic.urdf.xacro"/>
+  <xacro:add_world>
+    <origin xyz="0 0 0.2" rpy="0 0 0"/>
+  </xacro:add_world>
   <xacro:parallel_base_v0 parent="tool0"/>
   <xacro:parallel_grip_v0 prefix="right">
