Commit message: [modify] kinectの位置を修正

File: motoman_description/robots/sia5/sia5_with_parallel_and_kinectv2.urdf.xacro (robot description, xacro)
@@ -11,5 +11,5 @@
   <!-- Joint -->
   <joint name="joint_kinect2" type="fixed">
-	<origin xyz="1.3 0.0 0.6" rpy="0 ${20.0*M_PI/180.0} ${M_PI}" />
+	<origin xyz="1.0 0.0 0.3" rpy="0 ${30.0*M_PI/180.0} ${M_PI}" />
     <parent link="base_link"/>
     <child link="kinect2_link"/>
