Commit message: [Update]

File: motoman_description/robots/sia5/sia5_with_dhand_and_multi_kinect.urdf.xacro (robot description, xacro)
@@ -29,5 +29,5 @@
   <!-- Joint -->
   <joint name="joint_kinect_second" type="fixed">
-	<origin xyz="1.0013 1.2696 0.5348" rpy="-0.0249 0.2883 -2.0823" />
+	<origin xyz="0.9992 1.2708 0.5301" rpy="-0.0145 0.3292 -2.017" />
     <parent link="base_link"/>
     <child link="kinect_second_link"/>

Commit message: [modify] kinect first position & pose

File: motoman_description/robots/sia5/sia5_with_dhand_and_multi_kinect.urdf.xacro (robot description, xacro)
@@ -12,5 +12,6 @@
   <!-- Joint -->
   <joint name="joint_kinect_first" type="fixed">
-    <origin xyz="0.8794 -0.6445 0.5804" rpy="-0.035 0.3421 2.0509" />
+    <!-- <origin xyz="0.8794 -0.6445 0.5804" rpy="-0.035 0.3421 2.0509" /> -->
+	<origin xyz="1.17167 -0.738268 0.637113" rpy="-0.0710487 0.330165 2.40095" />
     <parent link="base_link"/>
     <child link="kinect_first_link"/>
@@ -29,5 +30,6 @@
   <!-- Joint -->
   <joint name="joint_kinect_second" type="fixed">
-	<origin xyz="1.4552 0.2663 0.4009" rpy="0.0327 0.4283 -2.9288" />
+	<!-- <origin xyz="1.4552 0.2663 0.4009" rpy="0.0327 0.4283 -2.9288" /> -->
+	<origin xyz="1.4552 0.3236 0.4009" rpy="0.0327 0.4283 -2.9288" />
     <parent link="base_link"/>
     <child link="kinect_second_link"/>
