Commit message: [modify] 新しいCADモデル用に変更
わけわかめ

File: motoman_description/robots/sia5/sia5.urdf.xacro (robot description, xacro)
@@ -3,6 +3,6 @@
   <!-- File Include -->
   <xacro:include filename="$(find motoman_description)/robots/sia5/sia5_basic.urdf.xacro" />
-  <xacro:add_world>
+  <xacro:root_link_v0 name="world">
     <origin xyz="0 0 0" rpy="0 0 0"/>
-  </xacro:add_world>
+  </xacro:root_link_v0>
 </robot>

File: motoman_description/robots/sia5/sia5_basic.urdf.xacro (robot description, xacro)
@@ -4,196 +4,121 @@
   <xacro:include filename="$(find motoman_description)/urdf/common.xacro" />
   <xacro:include filename="$(find motoman_description)/urdf/materials.xacro"/>
-  <xacro:include filename="$(find motoman_description)/urdf/sia5/body.urdf.xacro" />
-  <xacro:include filename="$(find motoman_description)/urdf/sia5/body.transmission.xacro"/>
-  <xacro:include filename="$(find motoman_description)/urdf/sia5/body.gazebo.xacro"/>
-  <!-- Mass -->
-  <property name="sum_mass" value="30.0" />
-  <!-- about mass rate -->
-  <property name="table_mass" value="40.0" />
-  <property name="base_rate" value="8.5" />
-  <property name="s_rate" value="7.7" />
-  <property name="l_rate" value="7.0" />
-  <property name="e_rate" value="1.2" />
-  <property name="u_rate" value="1.0" />
-  <property name="r_rate" value="0.9" />
-  <property name="b_rate" value="0.8" />
-  <property name="t_rate" value="0.5" />
+  <xacro:include filename="$(find motoman_description)/urdf/sia5/arm/arm.urdf.xacro" />
+  <xacro:include filename="$(find motoman_description)/urdf/sia5/base/base.urdf.xacro" />
   <!-- Hard ware limits -->
   <!-- Range limits -->
-  <xacro:property name="s_axis_upper_limit" value="${179.99999*M_PI/180.0*0.95}"/>
-  <xacro:property name="s_axis_lower_limit" value="-${s_axis_upper_limit}"/>
-  <xacro:property name="l_axis_upper_limit" value="${110.0*M_PI/180.0*0.95}"/>
-  <xacro:property name="l_axis_lower_limit" value="-${l_axis_upper_limit}"/>
-  <xacro:property name="e_axis_upper_limit" value="${170.0*M_PI/180.0*0.95}"/>
-  <xacro:property name="e_axis_lower_limit" value="-${e_axis_upper_limit}"/>
-  <xacro:property name="u_axis_upper_limit" value="${115.0*M_PI/180.0*0.95}"/>
-  <xacro:property name="u_axis_lower_limit" value="${-90.0*M_PI/180.0*0.95}"/>
-  <xacro:property name="r_axis_upper_limit" value="${179.99999*M_PI/180.0*0.95}"/>
-  <xacro:property name="r_axis_lower_limit" value="-${r_axis_upper_limit}"/>
-  <xacro:property name="b_axis_upper_limit" value="${110.0*M_PI/180.0*0.95}"/>
-  <xacro:property name="b_axis_lower_limit" value="-${b_axis_upper_limit}"/>
-  <xacro:property name="t_axis_upper_limit" value="${179.99999*M_PI/180.0*0.95}"/>
-  <xacro:property name="t_axis_lower_limit" value="-${t_axis_upper_limit}"/>
+  <xacro:property name="joint_s_upper_limit" value="${180*M_PI/180}"/>
+  <xacro:property name="joint_s_lower_limit" value="-${joint_s_upper_limit}"/>
+  <xacro:property name="joint_l_upper_limit" value="${110*M_PI/180}"/>
+  <xacro:property name="joint_l_lower_limit" value="-${joint_l_upper_limit}"/>
+  <xacro:property name="joint_e_upper_limit" value="${170*M_PI/180}"/>
+  <xacro:property name="joint_e_lower_limit" value="-${joint_e_upper_limit}"/>
+  <xacro:property name="joint_u_upper_limit" value="${115*M_PI/180}"/>
+  <xacro:property name="joint_u_lower_limit" value="${-90*M_PI/180}"/>
+  <xacro:property name="joint_r_upper_limit" value="${180*M_PI/180}"/>
+  <xacro:property name="joint_r_lower_limit" value="-${joint_r_upper_limit}"/>
+  <xacro:property name="joint_b_upper_limit" value="${110*M_PI/180}"/>
+  <xacro:property name="joint_b_lower_limit" value="-${joint_b_upper_limit}"/>
+  <xacro:property name="joint_t_upper_limit" value="${180*M_PI/180}"/>
+  <xacro:property name="joint_t_lower_limit" value="-${joint_t_upper_limit}"/>
   <!-- Velocity limits -->
-  <xacro:property name="s_axis_velocity_limit" value="${200.0*M_PI/180.0*0.95}"/>
-  <xacro:property name="l_axis_velocity_limit" value="${200.0*M_PI/180.0*0.95}"/>
-  <xacro:property name="e_axis_velocity_limit" value="${200.0*M_PI/180.0*0.95}"/>
-  <xacro:property name="u_axis_velocity_limit" value="${200.0*M_PI/180.0*0.95}"/>
-  <xacro:property name="r_axis_velocity_limit" value="${200.0*M_PI/180.0*0.95}"/>
-  <xacro:property name="b_axis_velocity_limit" value="${230.0*M_PI/180.0*0.95}"/>
-  <xacro:property name="t_axis_velocity_limit" value="${350.0*M_PI/180.0*0.95}"/>
-  <!-- Add macro -->
-  <xacro:macro name="add_world" params="*origin">
-    <link name="world"/>
-    <joint name="world" type="fixed">
-      <insert_block name="origin"/>
-      <parent link="world"/>
-      <child link="base_link"/>
-    </joint>
+  <xacro:property name="joint_s_velocity_limit" value="3.49"/>
+  <xacro:property name="joint_l_velocity_limit" value="3.49"/>
+  <xacro:property name="joint_e_velocity_limit" value="3.49"/>
+  <xacro:property name="joint_u_velocity_limit" value="3.49"/>
+  <xacro:property name="joint_r_velocity_limit" value="3.49"/>
+  <xacro:property name="joint_b_velocity_limit" value="4.01"/>
+  <xacro:property name="joint_t_velocity_limit" value="6.11"/>
+  <!-- Add Macro -->
+  <xacro:macro name="root_link_v0" params="name *joint_origin">
+    <link name="${name}"/>
+    <xacro:base_link_v0 parent="${name}">
+      <insert_block name="joint_origin"/>
+    </xacro:base_link_v0>
   </xacro:macro>
-  <!-- link -->
-  <xacro:link_box_v0 name="base_link" mass="${base_rate/sum_rate*sum_mass}"
-                     width="0.1665" depth="0.1976" height="0.1465"
-                     ox="-0.025918" oy="-0.000376" oz="0.076105" oroll="0" opitch="0" oyaw="0"/>
-  <xacro:link_cylinder_plus_box_v0 name="link_s"
-                                   ox="0" oy="0" oz="0" oroll="0" opitch="0" oyaw="0"
-                                   mass_cyl="${s_rate/sum_rate*sum_mass*0.2}"
-                                   radius_cyl="0.066" height_cyl="0.031"
-                                   mass_box="${s_rate/sum_rate*sum_mass*0.8}"
-                                   width_box="0.0851" depth_box="0.1" height_box="0.1823"/>
-  <xacro:link_cylinder_plus_box_v0 name="link_l"
-                                   ox="0" oy="-0.006" oz="0.15" oroll="${M_PI}" opitch="0" oyaw="0"
-                                   mass_cyl="${l_rate/sum_rate*sum_mass*0.4}"
-                                   radius_cyl="0.066" height_cyl="0.073"
-                                   mass_box="${l_rate/sum_rate*sum_mass*0.6}"
-                                   width_box="0.073" depth_box="0.1089" height_box="0.149"/>
-  <xacro:link_cylinder_plus_box_v0 name="link_e"
-                                   ox="0" oy="0" oz="0" oroll="0" opitch="0" oyaw="${-M_PI/2}"
-                                   mass_cyl="${e_rate/sum_rate*sum_mass*0.56}"
-                                   radius_cyl="0.0685" height_cyl="0.0661"
-                                   mass_box="${e_rate/sum_rate*sum_mass*0.44}"
-                                   width_box="0.1234" depth_box="0.063" height_box="0.1176"/>
-  <xacro:link_cylinder_plus_box_v0 name="link_u"
-                                   ox="0.008" oy="-0.06" oz="-0.131" oroll="${-M_PI}" opitch="${M_PI/2}" oyaw="0"
-                                   mass_cyl="${u_rate/sum_rate*sum_mass*0.48}"
-                                   radius_cyl="0.055" height_cyl="0.0698"
-                                   mass_box="${u_rate/sum_rate*sum_mass*0.52}"
-                                   width_box="0.13174" depth_box="0.068" height_box="0.104"/>
-  <xacro:link_cylinder_plus_box_v0 name="link_r"
-                                     ox="0" oy="0" oz="0" oroll="0" opitch="0" oyaw="${-M_PI/2}"
-                                     mass_cyl="${r_rate/sum_rate*sum_mass*0.25}"
-                                     radius_cyl="0.0525" height_cyl="0.038"
-                                     mass_box="${r_rate/sum_rate*sum_mass*0.75}"
-                                     width_box="0.0645" depth_box="0.084" height_box="0.1425"/>
-  <xacro:link_cylinder_plus_box_v0 name="link_b"
-                                     ox="0" oy="0.0045" oz="0.1365" oroll="${M_PI/2}" opitch="${-M_PI/2}" oyaw="0"
-                                     mass_cyl="${b_rate/sum_rate*sum_mass*0.55}"
-                                     radius_cyl="0.04" height_cyl="0.0948"
-                                     mass_box="${b_rate/sum_rate*sum_mass*0.45}"
-                                     width_box="0.0676" depth_box="0.076" height_box="0.0627"/>
-  <xacro:link_v1 name="link_t" mass="${t_rate/sum_rate*sum_mass}"
-                   ixx="0.003" ixy="0" ixz="0"
-                   iyy="0.003" iyz="0"
-                   izz="0.001"/>
-  <link name="tool0"/>
-  <!-- joint -->
-  <xacro:joint_v1 joint_name="joint_s"
-                  parent_name="base_link" child_name="link_s"
-                  ox="0" oy="0" oz="0.1765"
-                  roll="0" pitch="0" yaw="0"
-                  ax="0" ay="0" az="1"
-                  el="30.0"
-                  ll="${s_axis_lower_limit}" ul="${s_axis_upper_limit}"
-                  vl="${s_axis_velocity_limit}"
-                  skp="1" skv="1"
-                  sll="${s_axis_lower_limit}" sul="${s_axis_upper_limit}"/>
-  <xacro:joint_v1 joint_name="joint_l"
-                  parent_name="link_s" child_name="link_l"
-                  ox="0" oy="0.006" oz="0.136"
-                  roll="0" pitch="0" yaw="0"
-                  ax="0" ay="1" az="0"
-                  el="30.0"
-                  ll="${l_axis_lower_limit}" ul="${l_axis_upper_limit}"
-                  vl="${l_axis_velocity_limit}"
-                  skp="1" skv="1"
-                  sll="${l_axis_lower_limit}" sul="${l_axis_upper_limit}"/>
-  <xacro:joint_v1 joint_name="joint_e"
-                  parent_name="link_l" child_name="link_e"
-                  ox="0" oy="-0.006" oz="0.15"
-                  roll="0" pitch="0" yaw="0"
-                  ax="0" ay="0" az="1"
-                  el="30.0"
-                  ll="${e_axis_lower_limit}" ul="${e_axis_upper_limit}"
-                  vl="${e_axis_velocity_limit}"
-                  skp="1" skv="1"
-                  sll="${e_axis_lower_limit}" sul="${e_axis_upper_limit}"/>
-  <xacro:joint_v1 joint_name="joint_u"
-                  parent_name="link_e" child_name="link_u"
-                  ox="0.085" oy="-0.00826931" oz="0.12275299"
-                  roll="${M_PI/2.0}" pitch="0" yaw="0"
-                  ax="0" ay="0" az="1"
-                  el="30.0"
-                  ll="${u_axis_lower_limit}" ul="${u_axis_upper_limit}"
-                  vl="${u_axis_velocity_limit}"
-                  skp="1" skv="1"
-                  sll="${u_axis_lower_limit}" sul="${u_axis_upper_limit}"/>
-  <xacro:joint_v1 joint_name="joint_r"
-                  parent_name="link_u" child_name="link_r"
-                  ox="0.131" oy="0.06" oz="-0.008"
-                  roll="0" pitch="${M_PI/2}" yaw="0"
-                  ax="0" ay="0" az="-1"
-                  el="14.7"
-                  ll="${r_axis_lower_limit}" ul="${r_axis_upper_limit}"
-                  vl="${r_axis_velocity_limit}"
-                  skp="1" skv="1"
-                  sll="${r_axis_lower_limit}" sul="${r_axis_upper_limit}"/>
-  <xacro:joint_v1 joint_name="joint_b"
-                  parent_name="link_r" child_name="link_b"
-                  ox="-0.0045" oy="0" oz="0.139"
-                  roll="0" pitch="${-M_PI/2}" yaw="0"
-                  ax="0" ay="0" az="1"
-                  el="14.7"
-                  ll="${b_axis_lower_limit}" ul="${b_axis_upper_limit}"
-                  vl="${b_axis_velocity_limit}"
-                  skp="1" skv="1"
-                  sll="${b_axis_lower_limit}" sul="${b_axis_upper_limit}"/>
-  <xacro:joint_v1 joint_name="joint_t"
-                  parent_name="link_b" child_name="link_t"
-                  ox="0.1365" oy="0" oz="-0.0045"
-                  roll="${-M_PI/2}" pitch="0" yaw="0"
-                  ax="-1" ay="0" az="0"
-                  el="7.35"
-                  ll="${t_axis_lower_limit}" ul="${t_axis_upper_limit}"
-                  vl="${t_axis_velocity_limit}"
-                  skp="1" skv="1"
-                  sll="${t_axis_lower_limit}" sul="${t_axis_upper_limit}"/>
-  <joint name="joint_tool0" type="fixed">
-    <origin rpy="0 0 0" xyz="0.0115 0 0"/>
-    <parent link="link_t"/>
-    <child link="tool0"/>
-  </joint>
-  <!-- transmission -->
-  <xacro:simple_jp_trans_v0 name="transmission_s"
-                            joint_name="joint_s" actuator_name="motor_s"
-                            reduction="300"/>
-  <xacro:simple_jp_trans_v0 name="transmission_l"
-                            joint_name="joint_l" actuator_name="motor_l"
-                            reduction="300"/>
-  <xacro:simple_jp_trans_v0 name="transmission_e"
-                            joint_name="joint_e" actuator_name="motor_e"
-                            reduction="100"/>
-  <xacro:simple_jp_trans_v0 name="transmission_u"
-                            joint_name="joint_u" actuator_name="motor_u"
-                            reduction="50"/>
-  <xacro:simple_jp_trans_v0 name="transmission_r"
-                            joint_name="joint_r" actuator_name="motor_r"
-                            reduction="30"/>
-  <xacro:simple_jp_trans_v0 name="transmission_b"
-                            joint_name="joint_b" actuator_name="motor_b"
-                            reduction="30"/>
-  <xacro:simple_jp_trans_v0 name="transmission_t"
-                            joint_name="joint_t" actuator_name="motor_t"
-                            reduction="10"/>
-  <!-- gazebo -->
+  <!-- Add Link & Joint -->
+  <!-- Link S -->
+  <xacro:arm_v2 suffix="s" parent="base_link" mass="8.36956521739">
+    <origin xyz="0 0 0" rpy="0 0 0"/>
+    <inertia ixx="0.1285284" ixy="0" ixz="0"
+             iyy="0.127697251956" iyz="0" izz="0.0186623672464"/>
+    <origin xyz="0 0 0.1675" rpy="0 0 0"/>
+    <limit effort="30.0" lower="${joint_s_lower_limit}"
+           upper="${joint_s_upper_limit}" velocity="${joint_s_velocity_limit}"/>
+  </xacro:arm_v2>
+  <!-- Link L -->
+  <xacro:arm_v2 suffix="l" parent="link_s" mass="7.60869565217">
+    <origin rpy="3.14159274 0 0" xyz="0 -0.006 0.15"/>
+    <inertia ixx="0.12248884058" ixy="0" ixz="0"
+             iyy="0.117554616667" iyz="0" izz="0.0177495804348"/>
+    <origin xyz="0 0.0195 0.142" rpy="${-M_PI/2} 0 0"/>
+    <limit effort="30.0" lower="${joint_l_lower_limit}"
+           upper="${joint_l_upper_limit}" velocity="${joint_l_velocity_limit}"/>
+  </xacro:arm_v2>
+  <!-- Link E -->
+  <xacro:arm_v2 suffix="e" parent="link_l" mass="1.30434782609">
+    <origin rpy="0 0 -1.57079637" xyz="0 0 0"/>
+    <inertia ixx="0.0122899381739" ixy="0" ixz="0"
+             iyy="0.0117127787826" iyz="0" izz="0.00344401234783"/>
+    <origin xyz="0 -0.157 -0.0195" rpy="${M_PI/2} 0 0"/>
+    <limit effort="30.0" lower="${joint_e_lower_limit}"
+           upper="${joint_e_upper_limit}" velocity="${joint_e_velocity_limit}"/>
+  </xacro:arm_v2>
+  <!-- Link U -->
+  <xacro:arm_v2 suffix="u" parent="link_e" mass="1.08695652174">
+    <origin rpy="-3.14159274 1.57079637 0" xyz="0.008 -0.06 -0.131"/>
+    <inertia ixx="0.0110207115768" ixy="0" ixz="0"
+             iyy="0.00996803594202" iyz="0" izz="0.00214043853333"/>
+    <origin xyz="0.085 -0.017 0.113" rpy="0 ${M_PI/2} ${-M_PI/2}"/>
+    <limit effort="30.0" lower="${joint_u_lower_limit}"
+           upper="${joint_u_upper_limit}" velocity="${joint_u_velocity_limit}"/>
+  </xacro:arm_v2>
+  <!-- Link R -->
+  <xacro:arm_v2 suffix="r" parent="link_u" mass="0.978260869565">
+    <origin rpy="0 0 -1.57079637" xyz="0 0 0"/>
+    <inertia ixx="0.0108400832201" ixy="0" ixz="0"
+             iyy="0.010708873981" iyz="0" izz="0.00140456861413"/>
+    <origin xyz="-0.06 0.134 0.017" rpy="${M_PI/2} 0 0"/>
+    <limit effort="30.0" lower="${joint_r_lower_limit}"
+           upper="${joint_r_upper_limit}" velocity="${joint_r_velocity_limit}"/>
+  </xacro:arm_v2>
+  <!-- Link B -->
+  <xacro:arm_v2 suffix="b" parent="link_r" mass="0.869565217391">
+    <origin rpy="1.57079637 -1.57079637 0" xyz="0 0.0045 0.1365"/>
+    <inertia ixx="0.00814341869565" ixy="0" ixz="0"
+             iyy="0.00709473869565" iyz="0" izz="0.000736577391304"/>
+    <origin xyz="0 -0.0372 -0.136" rpy="${-M_PI/2} 0 0"/>
+    <limit effort="30.0" lower="${joint_b_lower_limit}"
+           upper="${joint_b_upper_limit}" velocity="${joint_b_velocity_limit}"/>
+  </xacro:arm_v2>
+  <!-- Link T -->
+  <xacro:arm_v2 suffix="t" parent="link_b" mass="0.54347826087">
+    <origin xyz="0 0 0" rpy="0 0 0"/>
+    <inertia ixx="0.003" ixy="0" ixz="0" iyy="0.003" iyz="0" izz="0.001"/>
+    <origin xyz="0 0.1365 0.0372" rpy="${M_PI/2} 0 0"/>
+    <limit effort="30.0" lower="${joint_t_lower_limit}"
+           upper="${joint_t_upper_limit}" velocity="${joint_t_velocity_limit}"/>
+  </xacro:arm_v2>
+  <!-- Link Tool -->
+  <xacro:link_tool_v0 parent="link_t">
+    <origin xyz="0 0 -0.011" rpy="${M_PI} ${M_PI/2} 0"/>
+  </xacro:link_tool_v0>
+  <!-- Add Transmission -->
+  <xacro:trans_v0 suffix="s" reduction="300"/>
+  <xacro:trans_v0 suffix="l" reduction="300"/>
+  <xacro:trans_v0 suffix="e" reduction="100"/>
+  <xacro:trans_v0 suffix="u" reduction="50"/>
+  <xacro:trans_v0 suffix="r" reduction="30"/>
+  <xacro:trans_v0 suffix="b" reduction="30"/>
+  <xacro:trans_v0 suffix="t" reduction="10"/>
+  <!-- Add Gazebo -->
+  <xacro:gazebo_v1 suffix="s"/>
+  <xacro:gazebo_v1 suffix="l"/>
+  <xacro:gazebo_v1 suffix="e"/>
+  <xacro:gazebo_v1 suffix="u"/>
+  <xacro:gazebo_v1 suffix="r"/>
+  <xacro:gazebo_v1 suffix="b"/>
+  <xacro:gazebo_v1 suffix="t"/>
+  <!-- Add Gazebo plugin -->
   <gazebo>
     <plugin name="gazebo_ros_control" filename="libgazebo_ros_control.so">
@@ -201,11 +126,3 @@
     </plugin>
   </gazebo>
-  <xacro:gazebo_link_v1 name="base_link"/>
-  <xacro:gazebo_link_v1 name="link_s"/>
-  <xacro:gazebo_link_v1 name="link_l"/>
-  <xacro:gazebo_link_v1 name="link_e"/>
-  <xacro:gazebo_link_v1 name="link_u"/>
-  <xacro:gazebo_link_v1 name="link_r"/>
-  <xacro:gazebo_link_v1 name="link_b"/>
-  <xacro:gazebo_link_v1 name="link_t"/>
 </robot>

File: motoman_description/robots/sia5/sia5_with_dhand.urdf.xacro (robot description, xacro)
@@ -2,13 +2,10 @@
 <robot name="sia5" xmlns:xacro="http://ros.org/wiki/xacro">
   <!-- File Include -->
-  <xacro:include filename="$(find motoman_description)/robots/sia5/sia5_basic.urdf.xacro"/>
+  <xacro:include filename="$(find motoman_description)/robots/sia5/sia5.urdf.xacro"/>
   <xacro:include filename="$(find dhand_description)/robots/dhand_adapted.urdf.xacro"/>
-  <xacro:add_world>
-    <origin xyz="0 0 0.2" rpy="0 0 0"/>
-  </xacro:add_world>
   <!-- Joint -->
   <joint name="dhand_adapter_joint" type="fixed">
 	<origin xyz="0 0 0" rpy="${M_PI} 0 0"/>
-	<parent link="tool0"/>
+	<parent link="tool_link"/>
 	<child link="dhand_adapter_link"/>
   </joint>
